File: hardware/ESP8266-PowerMonitor.sch (KiCad schematic (older format))
At the start: 5 parts, among them P1 CONN_01X15, P2 CONN_01X15, P3 CONN_01X02, P4 CONN_01X05

Commit message: Added the rest of wires + 1wire bus.
Parts:
- added P5, P?: CONN_01X03, symbol CONN_01X03
Connections:
- net at P2.15 (P15), R1.1: now also P4.4 (P4), P5.2 (P2), P?.1 (P1)
- net at P1.14 (P14): now also P4.1 (P1), P5.1 (P1), P?.3 (P3)
- net at P1.15 (P15): now also P4.5 (P5), P5.3 (P3)
Other:
- note added: "1Wire"
- note added: "3.3V\n"
Changed lines of the file:
@@
 LIBS:contrib
 LIBS:valves
+LIBS:ESP8266-PowerMonitor-cache
 EELAYER 25 0
 EELAYER END
@@
 $EndComp
 Wire Wire Line
-	7800 3400 7650 3400
+	7400 3400 7800 3400
 Wire Wire Line
 	7650 3400 7650 3550
@@
 Text Notes 6450 4300 0    60   ~ 0
 I2C
+$Comp
+L CONN_01X03 P5
+U 1 1 566A8677
+P 8000 4700
+F 0 "P5" H 8000 4900 50  0000 C CNN
+F 1 "CONN_01X03" V 8100 4700 50  0000 C CNN
+F 2 "" H 8000 4700 60  0000 C CNN
+F 3 "" H 8000 4700 60  0000 C CNN
+	1    8000 4700
+	1    0    0    -1
+$EndComp
+Wire Wire Line
+	7000 3300 7450 3300
+Wire Wire Line
+	7450 3300 7450 5000
+Wire Wire Line
+	7450 4600 7800 4600
+Wire Wire Line
+	7400 3400 7400 5200
+Wire Wire Line
+	7400 4700 7800 4700
+Connection ~ 7650 3400
+Wire Wire Line
+	7000 3400 7350 3400
+Wire Wire Line
+	7350 3400 7350 4800
+Wire Wire Line
+	7350 4800 7800 4800
+Text Notes 8150 4650 0    60   ~ 0
+GND
+Text Notes 8150 4750 0    60   ~ 0
+3.3V\n
+Text Notes 8150 4850 0    60   ~ 0
+5V
+Wire Wire Line
+	7000 4100 7450 4100
+Connection ~ 7450 4100
+Wire Wire Line
+	7000 4400 7400 4400
+Connection ~ 7400 4400
+Wire Wire Line
+	7000 4500 7350 4500
+Connection ~ 7350 4500
+$Comp
+L CONN_01X03 P?
+U 1 1 566A8D76
+P 6800 5100
+F 0 "P?" H 6800 5300 50  0000 C CNN
+F 1 "CONN_01X03" V 6900 5100 50  0000 C CNN
+F 2 "" H 6800 5100 60  0000 C CNN
+F 3 "" H 6800 5100 60  0000 C CNN
+	1    6800 5100
+	-1   0    0    1
+$EndComp
+Wire Wire Line
+	7400 5200 7000 5200
+Connection ~ 7400 4700
+Wire Wire Line
+	7450 5000 7000 5000
+Connection ~ 7450 4600
+Text Notes 6350 5150 0    60   ~ 0
+1Wire
 $EndSCHEMATC

Commit message: A few updates to the scheamtics.
Parts:
- P1, P2: footprint (none) -> Pin_Headers:Pin_Header_Straight_1x15
- P3: footprint (none) -> Pin_Headers:Pin_Header_Straight_1x02
- P4: footprint (none) -> Pin_Headers:Pin_Header_Straight_1x05
- P5: footprint (none) -> Pin_Headers:Pin_Header_Straight_1x03
- P6: renamed from P?; footprint (none) -> Pin_Headers:Pin_Header_Straight_1x03
Changed lines of the file:
@@
 F 0 "P2" H 8000 3500 50  0000 C CNN
 F 1 "CONN_01X15" V 8100 2700 50  0000 C CNN
-F 2 "" H 8000 2700 60  0000 C CNN
+F 2 "Pin_Headers:Pin_Header_Straight_1x15" H 8000 2700 60  0001 C CNN
 F 3 "" H 8000 2700 60  0000 C CNN
 	1    8000 2700
@@
 F 0 "P1" H 6800 3500 50  0000 C CNN
 F 1 "CONN_01X15" V 6900 2700 50  0000 C CNN
-F 2 "" H 6800 2700 60  0000 C CNN
+F 2 "Pin_Headers:Pin_Header_Straight_1x15" H 6800 2700 60  0001 C CNN
 F 3 "" H 6800 2700 60  0000 C CNN
 	1    6800 2700
@@
 F 0 "R1" V 7730 3700 50  0000 C CNN
 F 1 "220" V 7650 3700 50  0000 C CNN
-F 2 "" V 7580 3700 30  0000 C CNN
+F 2 "" V 7580 3700 30  0001 C CNN
 F 3 "" H 7650 3700 30  0000 C CNN
 	1    7650 3700
@@
 F 0 "P3" H 8000 4150 50  0000 C CNN
 F 1 "CONN_01X02" V 8100 4000 50  0000 C CNN
-F 2 "" H 8000 4000 60  0000 C CNN
+F 2 "Pin_Headers:Pin_Header_Straight_1x02" H 8000 4000 60  0001 C CNN
 F 3 "" H 8000 4000 60  0000 C CNN
 	1    8000 4000
@@
 F 0 "P4" H 6800 4600 50  0000 C CNN
 F 1 "CONN_01X05" V 6900 4300 50  0000 C CNN
-F 2 "" H 6800 4300 60  0000 C CNN
+F 2 "Pin_Headers:Pin_Header_Straight_1x05" H 6800 4300 60  0001 C CNN
 F 3 "" H 6800 4300 60  0000 C CNN
 	1    6800 4300
@@
 F 0 "P5" H 8000 4900 50  0000 C CNN
 F 1 "CONN_01X03" V 8100 4700 50  0000 C CNN
-F 2 "" H 8000 4700 60  0000 C CNN
+F 2 "Pin_Headers:Pin_Header_Straight_1x03" H 8000 4700 60  0001 C CNN
 F 3 "" H 8000 4700 60  0000 C CNN
 	1    8000 4700
@@
 Connection ~ 7350 4500
 $Comp
-L CONN_01X03 P?
+L CONN_01X03 P6
 U 1 1 566A8D76
 P 6800 5100
-F 0 "P?" H 6800 5300 50  0000 C CNN
+F 0 "P6" H 6800 5300 50  0000 C CNN
 F 1 "CONN_01X03" V 6900 5100 50  0000 C CNN
-F 2 "" H 6800 5100 60  0000 C CNN
+F 2 "Pin_Headers:Pin_Header_Straight_1x03" H 6800 5100 60  0001 C CNN
 F 3 "" H 6800 5100 60  0000 C CNN
 	1    6800 5100

Commit message: Almost done with the board.
Parts:
- removed P4: CONN_01X05, Pin_Headers:Pin_Header_Straight_1x05, symbol CONN_01X05
- added P4: CONN_01X03, Pin_Headers:Pin_Header_Straight_1x03, symbol CONN_01X03
- added R2: 4.7k, Resistors_ThroughHole:Resistor_Horizontal_RM10mm, symbol R
- P1, P2: footprint Pin_Headers:Pin_Header_Straight_1x15 -> Socket_Strips:Socket_Strip_Straight_1x15
- R1: footprint (none) -> Resistors_ThroughHole:Resistor_Horizontal_RM10mm
Connections:
- net at P2.2 (P2): now also P4.2 (P2)
- net at P2.4 (P4): now also R2.1
- net at P1.14 (P14), P5.1 (P1), P6.3 (P3): now also P4.1 (P1)
- net at P1.15 (P15), P5.3 (P3): now also P4.3 (P3)
- net at P6.2 (P2): now also R2.2
Other:
- note added: "GPIO0"
- note added: "GPIO5"
- note added: "PIR"
- note removed: "I2C"
Changed lines of the file:
@@
 F 0 "P2" H 8000 3500 50  0000 C CNN
 F 1 "CONN_01X15" V 8100 2700 50  0000 C CNN
-F 2 "Pin_Headers:Pin_Header_Straight_1x15" H 8000 2700 60  0001 C CNN
+F 2 "Socket_Strips:Socket_Strip_Straight_1x15" H 8000 2700 60  0001 C CNN
 F 3 "" H 8000 2700 60  0000 C CNN
 	1    8000 2700
@@
 F 0 "P1" H 6800 3500 50  0000 C CNN
 F 1 "CONN_01X15" V 6900 2700 50  0000 C CNN
-F 2 "Pin_Headers:Pin_Header_Straight_1x15" H 6800 2700 60  0001 C CNN
+F 2 "Socket_Strips:Socket_Strip_Straight_1x15" H 6800 2700 60  0001 C CNN
 F 3 "" H 6800 2700 60  0000 C CNN
 	1    6800 2700
@@
 F 0 "R1" V 7730 3700 50  0000 C CNN
 F 1 "220" V 7650 3700 50  0000 C CNN
-F 2 "" V 7580 3700 30  0001 C CNN
+F 2 "Resistors_ThroughHole:Resistor_Horizontal_RM10mm" V 7580 3700 30  0001 C CNN
 F 3 "" H 7650 3700 30  0000 C CNN
 	1    7650 3700
@@
 -
 $Comp
-L CONN_01X05 P4
-U 1 1 5664D204
-P 6800 4300
-F 0 "P4" H 6800 4600 50  0000 C CNN
-F 1 "CONN_01X05" V 6900 4300 50  0000 C CNN
-F 2 "Pin_Headers:Pin_Header_Straight_1x05" H 6800 4300 60  0001 C CNN
-F 3 "" H 6800 4300 60  0000 C CNN
-	1    6800 4300
-	-1   0    0    -1
-$EndComp
-Text Notes 6450 4300 0    60   ~ 0
-I2C
-$Comp
 L CONN_01X03 P5
 U 1 1 566A8677
@@
 Text Notes 8150 4850 0    60   ~ 0
 5V
-Wire Wire Line
-	7000 4100 7450 4100
-Connection ~ 7450 4100
-Wire Wire Line
-	7000 4400 7400 4400
-Connection ~ 7400 4400
-Wire Wire Line
-	7000 4500 7350 4500
-Connection ~ 7350 4500
 $Comp
 L CONN_01X03 P6
@@
 Text Notes 6350 5150 0    60   ~ 0
 1Wire
+Text Notes 8100 2350 0    60   ~ 0
+GPIO0
+$Comp
+L R R2
+U 1 1 566F3AF7
+P 7250 2650
+F 0 "R2" V 7330 2650 50  0000 C CNN
+F 1 "4.7k" V 7250 2650 50  0000 C CNN
+F 2 "Resistors_ThroughHole:Resistor_Horizontal_RM10mm" V 7180 2650 30  0001 C CNN
+F 3 "" H 7250 2650 30  0000 C CNN
+	1    7250 2650
+	1    0    0    -1
+$EndComp
+Wire Wire Line
+	7250 2500 7250 2300
+Wire Wire Line
+	7250 2300 7800 2300
+Wire Wire Line
+	7000 5100 7250 5100
+Wire Wire Line
+	7250 5100 7250 2800
+$Comp
+L CONN_01X03 P4
+U 1 1 566F3C3D
+P 6800 4150
+F 0 "P4" H 6800 4350 50  0000 C CNN
+F 1 "CONN_01X03" V 6900 4150 50  0000 C CNN
+F 2 "Pin_Headers:Pin_Header_Straight_1x03" H 6800 4150 60  0001 C CNN
+F 3 "" H 6800 4150 60  0000 C CNN
+	1    6800 4150
+	-1   0    0    1
+$EndComp
+Wire Wire Line
+	7000 4050 7350 4050
+Connection ~ 7350 4050
+Wire Wire Line
+	7000 4250 7450 4250
+Connection ~ 7450 4250
+Text Notes 8100 2150 0    60   ~ 0
+GPIO5
+Wire Wire Line
+	7800 2100 7150 2100
+Wire Wire Line
+	7150 2100 7150 4150
+Wire Wire Line
+	7150 4150 7000 4150
+Text Notes 6450 4200 0    60   ~ 0
+PIR
 $EndSCHEMATC

Commit message: Production prints.
Parts:
- P1: value CONN_01X15 -> CONN_LEFT
- P2: value CONN_01X15 -> CONN_RIGHT
- P3: value CONN_01X02 -> CONN_METER
- P4: value CONN_01X03 -> CONN_PIR
- P5: value CONN_01X03 -> CONN_POWER
- P6: value CONN_01X03 -> CONN_1WIRE
Connections:
- net at P3.2 (P2): now also R1.1; no longer P2.11 (P11)
- net GND: now reaches P2.14 (P14)
- net GND: now also P1.14 (P14), P4.1 (P1), P5.1 (P1), P6.1 (P1)
- net 3.3V: now reaches P2.15 (P15), P5.2 (P2)
- net 3.3V: now also P6.3 (P3), R1.2; no longer P6.1 (P1), R1.1
- net GPIO5: now reaches P2.2 (P2), P4.2 (P2)
- net at R2.1: now also P6.2 (P2); no longer P2.4 (P4)
- net 5V: now reaches P1.15 (P15), P4.3 (P3), P5.3 (P3)
- net GPIO15: now reaches P3.1 (P1)
- net GPIO15: now also P2.11 (P11); no longer R1.2
- net GPIO0: now reaches R2.2
- net GPIO0: now also P2.4 (P4); no longer P6.2 (P2)
Other:
- note removed: "3.3V\n"
- moved on the sheet: P3, P4, P5, P6, R1, R2
Changed lines of the file:
@@
 P 8000 2700
 F 0 "P2" H 8000 3500 50  0000 C CNN
-F 1 "CONN_01X15" V 8100 2700 50  0000 C CNN
+F 1 "CONN_RIGHT" V 8100 2700 50  0000 C CNN
 F 2 "Socket_Strips:Socket_Strip_Straight_1x15" H 8000 2700 60  0001 C CNN
 F 3 "" H 8000 2700 60  0000 C CNN
@@
 P 6800 2700
 F 0 "P1" H 6800 3500 50  0000 C CNN
-F 1 "CONN_01X15" V 6900 2700 50  0000 C CNN
+F 1 "CONN_LEFT" V 6900 2700 50  0000 C CNN
 F 2 "Socket_Strips:Socket_Strip_Straight_1x15" H 6800 2700 60  0001 C CNN
 F 3 "" H 6800 2700 60  0000 C CNN
@@
 L R R1
 U 1 1 5664D0EB
-P 7650 3700
-F 0 "R1" V 7730 3700 50  0000 C CNN
-F 1 "220" V 7650 3700 50  0000 C CNN
-F 2 "Resistors_ThroughHole:Resistor_Horizontal_RM10mm" V 7580 3700 30  0001 C CNN
-F 3 "" H 7650 3700 30  0000 C CNN
-	1    7650 3700
-	1    0    0    -1
+P 10050 4300
+F 0 "R1" V 10130 4300 50  0000 C CNN
+F 1 "220" V 10050 4300 50  0000 C CNN
+F 2 "Resistors_ThroughHole:Resistor_Horizontal_RM10mm" V 9980 4300 30  0001 C CNN
+F 3 "" H 10050 4300 30  0000 C CNN
+	1    10050 4300
+	0    1    1    0
 $EndComp
 $Comp
 L CONN_01X02 P3
 U 1 1 5664D153
-P 8000 4000
-F 0 "P3" H 8000 4150 50  0000 C CNN
-F 1 "CONN_01X02" V 8100 4000 50  0000 C CNN
-F 2 "Pin_Headers:Pin_Header_Straight_1x02" H 8000 4000 60  0001 C CNN
-F 3 "" H 8000 4000 60  0000 C CNN
-	1    8000 4000
-	1    0    0    -1
-$EndComp
-Wire Wire Line
-	7400 3400 7800 3400
-Wire Wire Line
-	7650 3400 7650 3550
-Wire Wire Line
-	7650 3850 7650 3950
-Wire Wire Line
-	7650 3950 7800 3950
-Wire Wire Line
-	7800 3000 7500 3000
-Wire Wire Line
-	7500 3000 7500 4050
-Wire Wire Line
-	7500 4050 7800 4050
-Text Notes 8150 4000 0    60   ~ 0
+P 10600 4250
+F 0 "P3" H 10600 4400 50  0000 C CNN
+F 1 "CONN_METER" V 10700 4250 50  0000 C CNN
+F 2 "Pin_Headers:Pin_Header_Straight_1x02" H 10600 4250 60  0001 C CNN
+F 3 "" H 10600 4250 60  0000 C CNN
+	1    10600 4250
+	1    0    0    -1
+$EndComp
+Text Notes 10800 4250 0    60   ~ 0
 +
-Text Notes 8150 4100 0    60   ~ 0
+Text Notes 10800 4350 0    60   ~ 0
 -
 $Comp
 L CONN_01X03 P5
 U 1 1 566A8677
-P 8000 4700
-F 0 "P5" H 8000 4900 50  0000 C CNN
-F 1 "CONN_01X03" V 8100 4700 50  0000 C CNN
-F 2 "Pin_Headers:Pin_Header_Straight_1x03" H 8000 4700 60  0001 C CNN
-F 3 "" H 8000 4700 60  0000 C CNN
-	1    8000 4700
-	1    0    0    -1
-$EndComp
-Wire Wire Line
-	7000 3300 7450 3300
-Wire Wire Line
-	7450 3300 7450 5000
-Wire Wire Line
-	7450 4600 7800 4600
-Wire Wire Line
-	7400 3400 7400 5200
-Wire Wire Line
-	7400 4700 7800 4700
-Connection ~ 7650 3400
-Wire Wire Line
-	7000 3400 7350 3400
-Wire Wire Line
-	7350 3400 7350 4800
-Wire Wire Line
-	7350 4800 7800 4800
-Text Notes 8150 4650 0    60   ~ 0
-GND
-Text Notes 8150 4750 0    60   ~ 0
-3.3V\n
-Text Notes 8150 4850 0    60   ~ 0
-5V
+P 10600 5050
+F 0 "P5" H 10600 5250 50  0000 C CNN
+F 1 "CONN_POWER" V 10700 5050 50  0000 C CNN
+F 2 "Pin_Headers:Pin_Header_Straight_1x03" H 10600 5050 60  0001 C CNN
+F 3 "" H 10600 5050 60  0000 C CNN
+	1    10600 5050
+	1    0    0    -1
+$EndComp
 $Comp
 L CONN_01X03 P6
 U 1 1 566A8D76
-P 6800 5100
-F 0 "P6" H 6800 5300 50  0000 C CNN
-F 1 "CONN_01X03" V 6900 5100 50  0000 C CNN
-F 2 "Pin_Headers:Pin_Header_Straight_1x03" H 6800 5100 60  0001 C CNN
-F 3 "" H 6800 5100 60  0000 C CNN
-	1    6800 5100
-	-1   0    0    1
-$EndComp
-Wire Wire Line
-	7400 5200 7000 5200
-Connection ~ 7400 4700
-Wire Wire Line
-	7450 5000 7000 5000
-Connection ~ 7450 4600
-Text Notes 6350 5150 0    60   ~ 0
+P 6150 4850
+F 0 "P6" H 6150 5050 50  0000 C CNN
+F 1 "CONN_1WIRE" V 6250 4850 50  0000 C CNN
+F 2 "Pin_Headers:Pin_Header_Straight_1x03" H 6150 4850 60  0001 C CNN
+F 3 "" H 6150 4850 60  0000 C CNN
+	1    6150 4850
+	1    0    0    -1
+$EndComp
+Text Notes 6300 4900 0    60   ~ 0
 1Wire
 Text Notes 8100 2350 0    60   ~ 0
@@
 L R R2
 U 1 1 566F3AF7
-P 7250 2650
-F 0 "R2" V 7330 2650 50  0000 C CNN
-F 1 "4.7k" V 7250 2650 50  0000 C CNN
-F 2 "Resistors_ThroughHole:Resistor_Horizontal_RM10mm" V 7180 2650 30  0001 C CNN
-F 3 "" H 7250 2650 30  0000 C CNN
-	1    7250 2650
-	1    0    0    -1
-$EndComp
-Wire Wire Line
-	7250 2500 7250 2300
-Wire Wire Line
-	7250 2300 7800 2300
-Wire Wire Line
-	7000 5100 7250 5100
-Wire Wire Line
-	7250 5100 7250 2800
+P 5700 4850
+F 0 "R2" V 5780 4850 50  0000 C CNN
+F 1 "4.7k" V 5700 4850 50  0000 C CNN
+F 2 "Resistors_ThroughHole:Resistor_Horizontal_RM10mm" V 5630 4850 30  0001 C CNN
+F 3 "" H 5700 4850 30  0000 C CNN
+	1    5700 4850
+	0    1    1    0
+$EndComp
 $Comp
 L CONN_01X03 P4
 U 1 1 566F3C3D
-P 6800 4150
-F 0 "P4" H 6800 4350 50  0000 C CNN
-F 1 "CONN_01X03" V 6900 4150 50  0000 C CNN
-F 2 "Pin_Headers:Pin_Header_Straight_1x03" H 6800 4150 60  0001 C CNN
-F 3 "" H 6800 4150 60  0000 C CNN
-	1    6800 4150
-	-1   0    0    1
-$EndComp
-Wire Wire Line
-	7000 4050 7350 4050
-Connection ~ 7350 4050
-Wire Wire Line
-	7000 4250 7450 4250
-Connection ~ 7450 4250
+P 6150 4150
+F 0 "P4" H 6227 4192 50  0000 L CNN
+F 1 "CONN_PIR" H 6227 4092 50  0000 L CNN
+F 2 "Pin_Headers:Pin_Header_Straight_1x03" H 6150 4150 60  0001 C CNN
+F 3 "" H 6150 4150 60  0000 C CNN
+	1    6150 4150
+	1    0    0    -1
+$EndComp
 Text Notes 8100 2150 0    60   ~ 0
 GPIO5
-Wire Wire Line
-	7800 2100 7150 2100
-Wire Wire Line
-	7150 2100 7150 4150
-Wire Wire Line
-	7150 4150 7000 4150
-Text Notes 6450 4200 0    60   ~ 0
+Text Notes 6350 4150 0    60   ~ 0
 PIR
+Text GLabel 8400 3550 2    60   Input ~ 0
+GND
+Text GLabel 6450 3550 0    60   Input ~ 0
+GND
+Text GLabel 8400 3700 2    60   Input ~ 0
+3.3V
+Wire Wire Line
+	8400 3700 7750 3700
+Wire Wire Line
+	7750 3700 7750 3400
+Wire Wire Line
+	7750 3400 7800 3400
+Wire Wire Line
+	8400 3550 7700 3550
+Wire Wire Line
+	7700 3550 7700 3300
+Wire Wire Line
+	7700 3300 7800 3300
+Text GLabel 9700 4150 0    60   Input ~ 0
+GPIO15
+Text GLabel 9700 4300 0    60   Input ~ 0
+3.3V
+Wire Wire Line
+	9700 4150 10400 4150
+Wire Wire Line
+	10400 4150 10400 4200
+Wire Wire Line
+	9700 4300 9900 4300
+Wire Wire Line
+	10200 4300 10400 4300
+Text GLabel 9800 4900 0    60   Input ~ 0
+GND
+Text GLabel 9800 5050 0    60   Input ~ 0
+3.3V
+Text GLabel 9800 5200 0    60   Input ~ 0
+5V
+Wire Wire Line
+	9800 4900 10400 4900
+Wire Wire Line
+	10400 4900 10400 4950
+Wire Wire Line
+	9800 5050 10400 5050
+Wire Wire Line
+	9800 5200 10400 5200
+Wire Wire Line
+	10400 5200 10400 5150
+Text GLabel 5600 4000 0    60   Input ~ 0
+GND
+Text GLabel 5600 4300 0    60   Input ~ 0
+5V
+Wire Wire Line
+	5600 4000 5950 4000
+Wire Wire Line
+	5950 4000 5950 4050
+Wire Wire Line
+	5600 4300 5950 4300
+Wire Wire Line
+	5950 4300 5950 4250
+Text GLabel 5600 4150 0    60   Input ~ 0
+GPIO5
+Wire Wire Line
+	5950 4150 5600 4150
+Text GLabel 5600 4700 0    60   Input ~ 0
+GND
+Text GLabel 5450 4850 0    60   Input ~ 0
+GPIO0
+Text GLabel 5600 5000 0    60   Input ~ 0
+3.3V
+Wire Wire Line
+	5600 5000 5950 5000
+Wire Wire Line
+	5950 5000 5950 4950
+Wire Wire Line
+	5600 4700 5950 4700
+Wire Wire Line
+	5950 4700 5950 4750
+Wire Wire Line
+	5450 4850 5550 4850
+Wire Wire Line
+	5850 4850 5950 4850
+Text GLabel 7700 2300 0    60   Input ~ 0
+GPIO0
+Text GLabel 7700 2100 0    60   Input ~ 0
+GPIO5
+Text GLabel 6450 3700 0    60   Input ~ 0
+5V
+Wire Wire Line
+	7000 3400 7050 3400
+Wire Wire Line
+	7050 3400 7050 3700
+Wire Wire Line
+	7050 3700 6450 3700
+Wire Wire Line
+	6450 3550 7100 3550
+Wire Wire Line
+	7100 3550 7100 3300
+Wire Wire Line
+	7100 3300 7000 3300
+Wire Wire Line
+	7700 2300 7800 2300
+Wire Wire Line
+	7700 2100 7800 2100
+Text GLabel 7700 3000 0    60   Input ~ 0
+GPIO15
+Wire Wire Line
+	7700 3000 7800 3000
 $EndSCHEMATC

Commit message: Updated schematics & PCB.
Connections:
- net 3.3V: now also P5.3 (P3), R2.1; no longer P5.2 (P2)
- net 5V: now also P5.2 (P2); no longer P5.3 (P3)
- net GPIO4: now reaches P2.3 (P3)
- net GPIO4: now also P6.2 (P2), R2.2
- net GPIO0: no longer names the net of P2.4 (P4)
- net GPIO0: no longer R2.2
Other:
- note added: "GPIO4"
- note removed: "GPIO0"
- moved on the sheet: R2
Changed lines of the file:
@@
 Text Notes 6300 4900 0    60   ~ 0
 1Wire
-Text Notes 8100 2350 0    60   ~ 0
-GPIO0
+Text Notes 8100 2250 0    60   ~ 0
+GPIO4
 $Comp
 L R R2
 U 1 1 566F3AF7
-P 5700 4850
-F 0 "R2" V 5780 4850 50  0000 C CNN
-F 1 "4.7k" V 5700 4850 50  0000 C CNN
-F 2 "Resistors_ThroughHole:Resistor_Horizontal_RM10mm" V 5630 4850 30  0001 C CNN
-F 3 "" H 5700 4850 30  0000 C CNN
-	1    5700 4850
-	0    1    1    0
+P 5700 5100
+F 0 "R2" V 5780 5100 50  0000 C CNN
+F 1 "4.7k" V 5700 5100 50  0000 C CNN
+F 2 "Resistors_ThroughHole:Resistor_Horizontal_RM10mm" V 5630 5100 30  0001 C CNN
+F 3 "" H 5700 5100 30  0000 C CNN
+	1    5700 5100
+	-1   0    0    1
 $EndComp
 $Comp
@@
 Text GLabel 9800 4900 0    60   Input ~ 0
 GND
+Text GLabel 9800 5200 0    60   Input ~ 0
+3.3V
 Text GLabel 9800 5050 0    60   Input ~ 0
-3.3V
-Text GLabel 9800 5200 0    60   Input ~ 0
 5V
 Wire Wire Line
@@
 Wire Wire Line
 	10400 4900 10400 4950
-Wire Wire Line
-	9800 5050 10400 5050
-Wire Wire Line
-	9800 5200 10400 5200
-Wire Wire Line
-	10400 5200 10400 5150
 Text GLabel 5600 4000 0    60   Input ~ 0
 GND
@@
 GND
 Text GLabel 5450 4850 0    60   Input ~ 0
-GPIO0
-Text GLabel 5600 5000 0    60   Input ~ 0
+GPIO4
+Text GLabel 5550 5300 0    60   Input ~ 0
 3.3V
-Wire Wire Line
-	5600 5000 5950 5000
-Wire Wire Line
-	5950 5000 5950 4950
 Wire Wire Line
 	5600 4700 5950 4700
 Wire Wire Line
 	5950 4700 5950 4750
-Wire Wire Line
-	5450 4850 5550 4850
-Wire Wire Line
-	5850 4850 5950 4850
-Text GLabel 7700 2300 0    60   Input ~ 0
-GPIO0
+Text GLabel 7700 2200 0    60   Input ~ 0
+GPIO4
 Text GLabel 7700 2100 0    60   Input ~ 0
 GPIO5
@@
 	7100 3300 7000 3300
 Wire Wire Line
-	7700 2300 7800 2300
-Wire Wire Line
 	7700 2100 7800 2100
 Text GLabel 7700 3000 0    60   Input ~ 0
@@
 Wire Wire Line
 	7700 3000 7800 3000
+Wire Wire Line
+	7700 2200 7800 2200
+Wire Wire Line
+	5450 4850 5950 4850
+Wire Wire Line
+	5700 4950 5700 4850
+Connection ~ 5700 4850
+Wire Wire Line
+	5550 5300 5950 5300
+Wire Wire Line
+	5700 5300 5700 5250
+Wire Wire Line
+	5950 5300 5950 4950
+Connection ~ 5700 5300
+Wire Wire Line
+	9800 5050 10400 5050
+Wire Wire Line
+	10400 5150 10400 5200
+Wire Wire Line
+	10400 5200 9800 5200
 $EndSCHEMATC

Commit message: Updated netlist and footprints.
Parts:
- added R3: 470, Resistors_ThroughHole:Resistor_Horizontal_RM10mm, symbol R
- R1: value 220 -> 470
Connections:
- net 3.3V: no longer R1.2
- net GND: now also R1.2
- net GPIO5: now also R3.2; no longer P4.2 (P2)
- net GPIO2: now reaches P2.5 (P5)
- net GPIO2: now also P3.1 (P1)
- net GPIO15: no longer names the net of P2.11 (P11)
- net GPIO15: no longer P3.1 (P1)
- new net: P4.2 (P2), R3.1
Changed lines of the file:
@@
 P 10050 4300
 F 0 "R1" V 10130 4300 50  0000 C CNN
-F 1 "220" V 10050 4300 50  0000 C CNN
+F 1 "470" V 10050 4300 50  0000 C CNN
 F 2 "Resistors_ThroughHole:Resistor_Horizontal_RM10mm" V 9980 4300 30  0001 C CNN
 F 3 "" H 10050 4300 30  0000 C CNN
@@
 	7700 3300 7800 3300
 Text GLabel 9700 4150 0    60   Input ~ 0
-GPIO15
+GPIO2
 Text GLabel 9700 4300 0    60   Input ~ 0
-3.3V
+GND
 Wire Wire Line
 	9700 4150 10400 4150
@@
 Wire Wire Line
 	10400 4900 10400 4950
-Text GLabel 5600 4000 0    60   Input ~ 0
+Text GLabel 5550 3900 0    60   Input ~ 0
 GND
-Text GLabel 5600 4300 0    60   Input ~ 0
+Text GLabel 5550 4400 0    60   Input ~ 0
 5V
-Wire Wire Line
-	5600 4000 5950 4000
-Wire Wire Line
-	5950 4000 5950 4050
-Wire Wire Line
-	5600 4300 5950 4300
-Wire Wire Line
-	5950 4300 5950 4250
-Text GLabel 5600 4150 0    60   Input ~ 0
+Text GLabel 5250 4150 0    60   Input ~ 0
 GPIO5
-Wire Wire Line
-	5950 4150 5600 4150
 Text GLabel 5600 4700 0    60   Input ~ 0
 GND
@@
 Wire Wire Line
 	7700 2100 7800 2100
-Text GLabel 7700 3000 0    60   Input ~ 0
-GPIO15
-Wire Wire Line
-	7700 3000 7800 3000
 Wire Wire Line
 	7700 2200 7800 2200
@@
 Wire Wire Line
 	10400 5200 9800 5200
+$Comp
+L R R3
+U 1 1 56891048
+P 5650 4150
+F 0 "R3" V 5455 4150 50  0000 C CNN
+F 1 "470" V 5555 4150 50  0000 C CNN
+F 2 "Resistors_ThroughHole:Resistor_Horizontal_RM10mm" V 5580 4150 50  0001 C CNN
+F 3 "" H 5650 4150 50  0000 C CNN
+	1    5650 4150
+	0    1    1    0
+$EndComp
+Wire Wire Line
+	5950 4150 5800 4150
+Wire Wire Line
+	5500 4150 5250 4150
+Wire Wire Line
+	5550 3900 5950 3900
+Wire Wire Line
+	5950 3900 5950 4050
+Wire Wire Line
+	5550 4400 5950 4400
+Wire Wire Line
+	5950 4400 5950 4250
+Text GLabel 7700 2400 0    60   Input ~ 0
+GPIO2
+Wire Wire Line
+	7700 2400 7800 2400
 $EndSCHEMATC

Commit message: Changed 4.7k resistor to 2.2k to facilitate greater 1 wire length.
Parts:
- R2: value 4.7k -> 2.2k
Changed lines of the file:
@@
 P 5700 5100
 F 0 "R2" V 5780 5100 50  0000 C CNN
-F 1 "4.7k" V 5700 5100 50  0000 C CNN
+F 1 "2.2k" V 5700 5100 50  0000 C CNN
 F 2 "Resistors_ThroughHole:Resistor_Horizontal_RM10mm" V 5630 5100 30  0001 C CNN
 F 3 "" H 5700 5100 30  0000 C CNN
