File: hardware/ESP8266-PowerMonitor.sch (KiCad schematic (older format))
At the start: 9 parts, among them P1 CONN_LEFT, P2 CONN_RIGHT, P3 CONN_METER, P4 CONN_PIR, P5 CONN_POWER, P6 CONN_1WIRE

Commit message: Redesigned the board.
Parts:
- removed P1: CONN_LEFT, Socket_Strips:Socket_Strip_Straight_1x15, symbol CONN_01X15
- removed P2: CONN_RIGHT, Socket_Strips:Socket_Strip_Straight_1x15, symbol CONN_01X15
- removed P3: CONN_METER, Pin_Headers:Pin_Header_Straight_1x02, symbol CONN_01X02
- removed P4: CONN_PIR, Pin_Headers:Pin_Header_Straight_1x03, symbol CONN_01X03
- removed P5: CONN_POWER, Pin_Headers:Pin_Header_Straight_1x03, symbol CONN_01X03
- removed P6: CONN_1WIRE, Pin_Headers:Pin_Header_Straight_1x03, symbol CONN_01X03
- removed R1, R3: 470, Resistors_ThroughHole:Resistor_Horizontal_RM10mm, symbol R
- removed R2: 2.2k, Resistors_ThroughHole:Resistor_Horizontal_RM10mm, symbol R
- added C1: 0.1uF, Capacitor_SMD:C_1206_3216Metric_Pad1.42x1.75mm_HandSolder, symbol Device:C
- added C2: 10uF, Capacitor_SMD:CP_Elec_4x5.3, symbol Device:CP
- added C3: 100nF, Capacitor_SMD:C_1206_3216Metric_Pad1.42x1.75mm_HandSolder, symbol Device:C
- added F1: 100mA, Fuse:Fuse_1206_3216Metric_Pad1.42x1.75mm_HandSolder, symbol Device:Polyfuse
- added J1: CONN_PULSE, Connector_PinHeader_2.54mm:PinHeader_1x02_P2.54mm_Vertical, symbol Connector:Conn_01x02_Male
- added J2: CONN_PROG, Connector_PinHeader_2.54mm:PinHeader_1x05_P2.54mm_Vertical, symbol Connector:Conn_01x05_Male
- added J3: CONN_AC, TerminalBlock:TerminalBlock_bornier-2_P5.08mm, symbol Connector:Conn_01x02_Male
- added J4: CONN_TEMP, Connector_PinHeader_2.54mm:PinHeader_1x03_P2.54mm_Vertical, symbol Connector:Conn_01x03_Male
- added JP1: 3.3V BYPASS, Jumper:SolderJumper-2_P1.3mm_Open_TrianglePad1.0x1.5mm, symbol Jumper:SolderJumper_2_Open
- added PS1: HLK-PM03, Converter_ACDC:Converter_ACDC_HiLink_HLK-PMxx, symbol Converter_ACDC:HLK-PM03
- added R1, R2, R4, R5, R6: 10k, Resistor_SMD:R_1206_3216Metric_Pad1.42x1.75mm_HandSolder, symbol Device:R
- added R3: 470, Resistor_SMD:R_1206_3216Metric_Pad1.42x1.75mm_HandSolder, symbol Device:R
- added SW1: SW_RESET, Button_Switch_SMD:SW_Push_1P1T_NO_6x6mm_H9.5mm, symbol Switch:SW_DIP_x01
- added U1: AMS1117-3.3, Package_TO_SOT_SMD:SOT-223-3_TabPin2, symbol Regulator_Linear:AMS1117-3.3
- added U2: ESP-12F, RF_Module:ESP-12E, symbol RF_Module:ESP-12F
Connections:
- net GND: now also C1.2, C2.2, C3.2, J1.2 (Pin_2), J2.1 (Pin_1), J4.2 (Pin_2), PS1.3 (-Vout), R6.1, SW1.2, U1.1 (GND), U2.15 (GND)
- new net: R1.1, SW1.1, U2.1 (~RST)
- new net: R6.2, U2.16 (GPIO15)
- new net: R5.2, U2.17 (GPIO2)
- new net: R3.1, U2.19 (GPIO4)
- new net: R2.2, U2.3 (EN)
- new net: C1.1, JP1.1 (A), PS1.4 (+Vout), U1.3 (VI)
- new net: F1.1, PS1.1 (AC/L)
- new net +3.3V: C2.1, C3.1, J2.5 (Pin_5), J4.3 (Pin_3), JP1.2 (B), R1.2, R2.1, R4.1, R5.1, U1.2 (VO), U2.8 (VCC)
- new net AC-L: F1.2, J3.2 (Pin_2)
- new net AC-N: J3.1 (Pin_1), PS1.2 (AC/N)
- new net DS18B20_DQ: J4.1 (Pin_1), U2.20 (GPIO5)
- new net PULSE: J1.1 (Pin_1), R3.2
- new net RXD: J2.3 (Pin_3), U2.21 (GPIO3/RXD)
- new net TXD: J2.4 (Pin_4), U2.22 (GPIO1/TXD)
- new net _PROG: J2.2 (Pin_2), R4.2, U2.18 (GPIO0)
- no-connect marks 0 -> 11
Other:
- note removed: "+"
- note removed: "-"
- note removed: "1Wire"
- note removed: "3.3V"
- note removed: "5V"
- note removed: "GND"
- note removed: "GPIO15\n"
- note removed: "GPIO4"
- note removed: "GPIO5"
- note removed: "PIR"
